File: cob/cob.brd (EAGLE design)
At the start: 75.8 x 67.1 mm, 36 parts

Commit message: fixed connections to cob board
Connections:
- net N$34 renamed XLAT
- net N$35 renamed GSCLK
- net N$37 renamed SOUT
- net N$6 renamed BLANK
- net N$7 renamed SCLK
- net N$8 renamed SIN
Changed lines of the file:
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@@
 <wire x1="53.05020625" y1="19.326628125" x2="52.585625" y2="19.326628125" width="0.254" layer="1"/>
 </signal>
-<signal name="N$6">
+<signal name="BLANK">
 <contactref element="U$1" pad="P$31"/>
 <contactref element="R2" pad="1"/>
@@
 <wire x1="50.893984375" y1="18.427703125" x2="50.175159375" y2="18.427703125" width="0.254" layer="16"/>
 </signal>
-<signal name="N$7">
+<signal name="SCLK">
 <contactref element="U$1" pad="P$1"/>
 <contactref element="U$2" pad="P$1"/>
@@
 <wire x1="41.395659375" y1="43.6156" x2="41.395659375" y2="41.8846" width="0.254" layer="1"/>
 </signal>
-<signal name="N$8">
+<signal name="SIN">
 <contactref element="U$1" pad="P$2"/>
 <contactref element="U$3" pad="P$5"/>
@@
 <wire x1="54.5566625" y1="14.38148125" x2="52.67451875" y2="15.5575" width="0.254" layer="16"/>
 </signal>
-<signal name="N$34">
+<signal name="XLAT">
 <contactref element="U$1" pad="P$32"/>
 <contactref element="U$2" pad="P$32"/>
@@
 <wire x1="30.48761875" y1="17.45488125" x2="26.629359375" y2="21.313140625" width="0.254" layer="16"/>
 </signal>
-<signal name="N$35">
+<signal name="GSCLK">
 <contactref element="U$1" pad="P$24"/>
 <contactref element="U$2" pad="P$24"/>
@@
 <wire x1="51.996340625" y1="26.4566375" x2="55.13831875" y2="23.314659375" width="0.254" layer="16"/>
 </signal>
-<signal name="N$37">
+<signal name="SOUT">
 <contactref element="U$2" pad="P$23"/>
 <contactref element="U$3" pad="P$2"/>
