File: spinner/spinner.sch (EAGLE design)
At the start: 50 parts, among them U2 ADXL330, Y1 16M

Commit message: fixed connections to cob board
Connections:
- removed net D5: U$7.PC6
- removed net D6: U$7.PD7(ADC10)
- removed net D8: U$7.PB4(ADC11)
- removed net D9: R11.1, U$7.D+, U$7.PB5(ADC12)
- new net D5/BLANK: U$7.PC6, U$8.P$2, U$9.P$2
- new net D6/SCLK: U$7.PD7(ADC10), U$8.P$3, U$9.P$3
- new net D7/SIN: U$8.P$4
- new net D8/XLAT: U$7.PB4(ADC11), U$8.P$5, U$9.P$5
- new net D9/GSCLK: R11.1, U$7.D+, U$7.PB5(ADC12), U$8.P$6, U$9.P$6
- new net SOUT: U$8.P$7, U$9.P$4
- net GND: now also U$8.P$8, U$9.P$8
- net VCC: now also U$8.P$1, U$9.P$1
Other:
- note added: "ACCELEROMETER"
- note added: "ATMEGA W/ USB PROGRAMMING"
- note added: "COB_BOTTOM"
- note added: "COB_TOP"
- note added: "LI ION CHERGER"
- note added: "MAIN POWER"
- note added: "SETTING SELECT"
- moved on the sheet: BAT+, BAT-, BAT2+, BAT2-, BAT3+, BAT3-, C4, C5, C6, C7, C8, C9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

Commit message: laid out traces on spinner brd
Connections:
- removed net D7: U$7.PE6
- removed net NC: U$2.P$4
- net 3.7+: now also C1.2, C9.2, D3.C, D4.C, R12.2, U$8.P$1, U$9.P$1, U2.VS, U2.VS@1
- net BAT+: now also U$2.P$3
- net D4: now also U$2.P$4; no longer U$2.P$3
- net D7/SIN: now also U$7.PE6
- net N$1: now also U$7.XTAL1
- net N$2: now also U$7.XTAL2
- net VCC: no longer C1.2, C9.2, D3.C, D4.C, R12.2, U$2.P$2, U$8.P$1, U$9.P$1, U2.VS, U2.VS@1
Other:
- moved on the sheet: D4, R7
